Commit message: Calibrate left arm URDF zero pose from RViz reference

File: remote_xiaogong_kaixuan/model/robot.urdf (robot description, URDF)
Before this commit: robot kaixuan1, 18 links, 17 joints
Joints:
- joint left_joint1: origin xyz=0 0.20995 -0.049457 rpy=-5.551115123125783e-16 1.3963 1.570803673205103 -> xyz=0 0.20995 -0.049457 rpy=1.2048263465734849e-16 -1.3963000000000005 -1.5707889803846902
- joint left_joint2: origin xyz=0 0 0.0727 rpy=1.5708 -1.5708 0 -> xyz=0 0 0.0727 rpy=1.5707926535986432 1.5707926536057681 1.5112462392383912e-11
- joint left_joint3: origin xyz=0 -0.1386 -0.0055244 rpy=1.5708 0 0 -> xyz=0 -0.1386 -0.0055244 rpy=1.570800027585129 0.12217304763877479 4.5101287572180343e-07
- joint left_joint4: origin xyz=0.00815 -0.003 0.19985 rpy=0 -1.5708 3.141592653589793 -> xyz=0.00815 -0.003 0.19985 rpy=-1.570802163575582 -0.89011791850877753 -1.5707917907643592
- joint left_joint5: origin xyz=0.15445 -0.005 -0.00815 rpy=0 1.5708 0 -> xyz=0.15445 -0.005 -0.00815 rpy=3.1415926535564531 -1.5707926536359933 3.3340005926160826e-11
- joint left_joint6: origin xyz=0 0 0.08405 rpy=0 -1.5708 0 -> xyz=0 0 0.08405 rpy=1.5708088902716077 -1.2740903539337951 -1.5708083413074267
- joint left_joint7: origin xyz=0.08945 0 0 rpy=0 1.5708 0 -> xyz=0.08945 0 0 rpy=-1.5708314675114721 1.4660765716110533 -1.5708312750069502

File: xiaogong_kaixuan/src/xiaogong_kaixuan/urdf/xiaogong-kaixuan.urdf (robot description, URDF)
Before this commit: robot xiaogong-kaixuan, 18 links, 17 joints
Joints:
- joint left_joint1: origin xyz=0 0.20995 -0.049457 rpy=-5.551115123125783e-16 1.3963 1.570803673205103 -> xyz=0 0.20995 -0.049457 rpy=1.2048263465734849e-16 -1.3963000000000005 -1.5707889803846902
- joint left_joint2: origin xyz=0 0 0.0727 rpy=1.5708 -1.5708 0 -> xyz=0 0 0.0727 rpy=1.5707926535986432 1.5707926536057681 1.5112462392383912e-11
- joint left_joint3: origin xyz=0 -0.1386 -0.0055244 rpy=1.5708 0 0 -> xyz=0 -0.1386 -0.0055244 rpy=1.570800027585129 0.12217304763877479 4.5101287572180343e-07
- joint left_joint4: origin xyz=0.00815 -0.003 0.19985 rpy=0 -1.5708 3.141592653589793 -> xyz=0.00815 -0.003 0.19985 rpy=-1.570802163575582 -0.89011791850877753 -1.5707917907643592
- joint left_joint5: origin xyz=0.15445 -0.005 -0.00815 rpy=0 1.5708 0 -> xyz=0.15445 -0.005 -0.00815 rpy=3.1415926535564531 -1.5707926536359933 3.3340005926160826e-11
- joint left_joint6: origin xyz=0 0 0.08405 rpy=0 -1.5708 0 -> xyz=0 0 0.08405 rpy=1.5708088902716077 -1.2740903539337951 -1.5708083413074267
- joint left_joint7: origin xyz=0.08945 0 0 rpy=0 1.5708 0 -> xyz=0.08945 0 0 rpy=-1.5708314675114721 1.4660765716110533 -1.5708312750069502

Commit message: Calibrate left arm encoder offsets and restore URDF geometry

File: remote_xiaogong_kaixuan/model/robot.urdf (robot description, URDF)
Before this commit: robot kaixuan1, 18 links, 17 joints
Joints:
- joint left_joint1: origin xyz=0 0.20995 -0.049457 rpy=1.2048263465734849e-16 -1.3963000000000005 -1.5707889803846902 -> xyz=0 0.20995 -0.049457 rpy=-5.551115123125783e-16 1.3963 1.570803673205103
- joint left_joint2: origin xyz=0 0 0.0727 rpy=1.5707926535986432 1.5707926536057681 1.5112462392383912e-11 -> xyz=0 0 0.0727 rpy=1.5708 -1.5708 0
- joint left_joint3: origin xyz=0 -0.1386 -0.0055244 rpy=1.570800027585129 0.12217304763877479 4.5101287572180343e-07 -> xyz=0 -0.1386 -0.0055244 rpy=1.5708 0 0
- joint left_joint4: origin xyz=0.00815 -0.003 0.19985 rpy=-1.570802163575582 -0.89011791850877753 -1.5707917907643592 -> xyz=0.00815 -0.003 0.19985 rpy=0 -1.5708 3.141592653589793
- joint left_joint5: origin xyz=0.15445 -0.005 -0.00815 rpy=3.1415926535564531 -1.5707926536359933 3.3340005926160826e-11 -> xyz=0.15445 -0.005 -0.00815 rpy=0 1.5708 0
- joint left_joint6: origin xyz=0 0 0.08405 rpy=1.5708088902716077 -1.2740903539337951 -1.5708083413074267 -> xyz=0 0 0.08405 rpy=0 -1.5708 0
- joint left_joint7: origin xyz=0.08945 0 0 rpy=-1.5708314675114721 1.4660765716110533 -1.5708312750069502 -> xyz=0.08945 0 0 rpy=0 1.5708 0

File: xiaogong_kaixuan/src/xiaogong_kaixuan/urdf/xiaogong-kaixuan.urdf (robot description, URDF)
Before this commit: robot xiaogong-kaixuan, 18 links, 17 joints
Joints:
- joint left_joint1: origin xyz=0 0.20995 -0.049457 rpy=1.2048263465734849e-16 -1.3963000000000005 -1.5707889803846902 -> xyz=0 0.20995 -0.049457 rpy=-5.551115123125783e-16 1.3963 1.570803673205103
- joint left_joint2: origin xyz=0 0 0.0727 rpy=1.5707926535986432 1.5707926536057681 1.5112462392383912e-11 -> xyz=0 0 0.0727 rpy=1.5708 -1.5708 0
- joint left_joint3: origin xyz=0 -0.1386 -0.0055244 rpy=1.570800027585129 0.12217304763877479 4.5101287572180343e-07 -> xyz=0 -0.1386 -0.0055244 rpy=1.5708 0 0
- joint left_joint4: origin xyz=0.00815 -0.003 0.19985 rpy=-1.570802163575582 -0.89011791850877753 -1.5707917907643592 -> xyz=0.00815 -0.003 0.19985 rpy=0 -1.5708 3.141592653589793
- joint left_joint5: origin xyz=0.15445 -0.005 -0.00815 rpy=3.1415926535564531 -1.5707926536359933 3.3340005926160826e-11 -> xyz=0.15445 -0.005 -0.00815 rpy=0 1.5708 0
- joint left_joint6: origin xyz=0 0 0.08405 rpy=1.5708088902716077 -1.2740903539337951 -1.5708083413074267 -> xyz=0 0 0.08405 rpy=0 -1.5708 0
- joint left_joint7: origin xyz=0.08945 0 0 rpy=-1.5708314675114721 1.4660765716110533 -1.5708312750069502 -> xyz=0.08945 0 0 rpy=0 1.5708 0
